Commit message: modify the my_robot.gazebo & xacro for RGBD camera

File: my_robot/urdf/my_robot_saved.xacro (robot description, xacro)
@@ -16,5 +16,30 @@
     <axis xyz="0 1 0" rpy="0 0 0"/>
   </joint>
-    <!-- Joint RGBD camera -->
+  <!-- Joint Chassis-Lidar(Hokuyo) -->
+  <joint name="hokuyo_joint" type="fixed">
+    <origin xyz="0.15 0 0.1" rpy="0 0 0" />
+    <parent link="chassis"/>
+    <child link="hokuyo"/>
+    <axis xyz="0 1 0" rpy="0 0 0"/>
+  </joint>
+  <!-- Joint Chassis-LeftWheel -->
+  <joint name="left_wheel_hinge" type="continuous">
+    <origin xyz="0 0.15 0" rpy="0 0 0"/>
+    <parent link="chassis"/>
+    <child link="left_wheel"/>
+    <axis xyz="0 1 0" rpy="0 0 0"/>
+    <limit effort="10000" velocity="1000"/>
+    <dynamics damping="1.0" friction="1.0"/>
+  </joint>
+  <!-- Joint Chassis-RightWheel -->
+  <joint name="right_wheel_hinge" type="continuous">
+    <origin xyz="0 -0.15 0" rpy="0 0 0"/>
+    <parent link="chassis"/>
+    <child link="right_wheel"/>
+    <axis xyz="0 1 0" rpy="0 0 0"/>
+    <limit effort="10000" velocity="1000"/>
+    <dynamics damping="1.0" friction="1.0"/>
+  </joint>
+  <!-- Joint RGBD camera -->
   <joint name="camera_optical_joint" type="fixed">
     <origin xyz="0 0 0" rpy="-1.5707 0 -1.5707"/>
@@ -22,29 +47,4 @@
     <child link="camera_link_optical"/>
   </joint>
-  <!-- Joint Chassis-Lidar(Hokuyo) -->
-  <joint name="hokuyo_joint" type="fixed">
-    <origin xyz="0.15 0 0.1" rpy="0 0 0" />
-    <parent link="chassis"/>
-    <child link="hokuyo"/>
-    <axis xyz="0 1 0" rpy="0 0 0"/>
-  </joint>
-  <!-- Joint Chassis-LeftWheel -->
-  <joint name="left_wheel_hinge" type="continuous">
-    <origin xyz="0 0.15 0" rpy="0 0 0"/>
-    <parent link="chassis"/>
-    <child link="left_wheel"/>
-    <axis xyz="0 1 0" rpy="0 0 0"/>
-    <limit effort="10000" velocity="1000"/>
-    <dynamics damping="1.0" friction="1.0"/>
-  </joint>
-  <!-- Joint Chassis-RightWheel -->
-  <joint name="right_wheel_hinge" type="continuous">
-    <origin xyz="0 -0.15 0" rpy="0 0 0"/>
-    <parent link="chassis"/>
-    <child link="right_wheel"/>
-    <axis xyz="0 1 0" rpy="0 0 0"/>
-    <limit effort="10000" velocity="1000"/>
-    <dynamics damping="1.0" friction="1.0"/>
-  </joint>
   <!-- Chassis -->
   <link name='chassis'>
