Commit message: Add sensors

File: my_robot/urdf/my_robot.xacro (robot description, xacro)
@@ -2,4 +2,5 @@
 <robot name="my_robot" xmlns:xacro="http://www.ros.org/wiki/xacro">
   <link name="robot_footprint"></link>
+  <!-- Joint FootPrint-Chassis -->
   <joint name="robot_footprint_joint" type="fixed">
     <origin xyz="0 0 0" rpy="0 0 0" />
@@ -7,4 +8,19 @@
     <child link="chassis" />
   </joint>
+  <!-- Joint Chassis-Camera -->
+  <joint name="camera_joint" type="fixed">
+    <origin xyz="0.2 0 0" rpy="0 0 0" />
+    <parent link="chassis"/>
+    <child link="camera" />
+    <axis xyz="0 1 0" rpy="0 0 0"/>
+  </joint>
+  <!-- Joint Chassis-Lidar(Hokuyo) -->
+  <joint name="hokuyo_joint" type="fixed">
+    <origin xyz="0.15 0 0.1" rpy="0 0 0" />
+    <parent link="chassis"/>
+    <child link="hokuyo"/>
+    <axis xyz="0 1 0" rpy="0 0 0"/>
+  </joint>
+  <!-- Joint Chassis-LeftWheel -->
   <joint type="continuous" name="left_wheel_hinge">
     <origin xyz="0 0.15 0" rpy="0 0 0"/>
@@ -15,4 +31,5 @@
     <dynamics damping="1.0" friction="1.0"/>
   </joint>
+  <!-- Joint Chassis-RightWheel -->
   <joint type="continuous" name="right_wheel_hinge">
     <origin xyz="0 -0.15 0" rpy="0 0 0"/>
@@ -125,3 +142,54 @@
   </link>
   <!-- End of the Right Wheel -->
+  <!-- Camera -->
+  <link name='camera'>
+    <inertial>
+      <mass value="0.1"/>
+      <origin xyz="0 0 0" rpy="0 0 0"/>
+      <box_inertia m="0.1" x="0.05" y="0.05" z="0.05"/>
+      <inertia
+          ixx="1e-6" ixy="0" ixz="0"
+          iyy="1e-6" iyz="0"
+          izz="1e-6"
+      />
+    </inertial>
+    <collision name='camera_collision'>
+      <origin xyz="0 0 0" rpy="0 0 0"/>
+      <geometry>
+        <box size="0.05 0.05 0.05"/>
+      </geometry>
+    </collision>
+    <visual name='camera_visual'>
+      <origin xyz="0 0 0" rpy="0 0 0"/>
+      <geometry>
+        <box size="0.05 0.05 0.05"/>
+      </geometry>
+    </visual>
+  </link>
+  <!-- End of the camera -->
+  <!-- Lidar(Hokuyo) -->
+  <link name='hokuyo'>
+    <inertial>
+      <mass value="1e-5"/>
+      <origin xyz="0 0 0" rpy="0 0 0"/>
+      <inertia
+          ixx="1e-6" ixy="0" ixz="0"
+          iyy="1e-6" iyz="0"
+          izz="1e-6"
+      />
+    </inertial>
+    <collision name='camera_collision'>
+      <origin xyz="0 0 0" rpy="0 0 0"/>
+      <geometry>
+        <box size="0.1 0.1 0.1"/>
+      </geometry>
+    </collision>
+    <visual name='camera_visual'>
+      <origin xyz="0 0 0" rpy="0 0 0"/>
+      <geometry>
+	<mesh filename="package://my_robot/meshes/hokuyo.dae"/>
+      </geometry>
+    </visual>
+  </link>
+  <!-- End of the Hokuyo -->
 </robot>

Commit message: Add material

File: my_robot/urdf/my_robot.xacro (robot description, xacro)
@@ -193,3 +193,17 @@
   </link>
   <!-- End of the Hokuyo -->
+  <!-- Color configuration -->
+  <gazebo reference="left_wheel">
+    <material>Gazebo/FlatBlack</material>
+  </gazebo>
+  <gazebo reference="right_wheel">
+    <material>Gazebo/FlatBlack</material>
+  </gazebo>
+  <gazebo reference="chassis">
+    <material>Gazebo/Indigo</material>
+  </gazebo>
+  <gazebo reference="camera">
+    <material>Gazebo/FlatBlack</material>
+  </gazebo>
+  <!-- End of the color configuration -->
 </robot>

Commit message: New world file and Control Plugin

File: my_robot/urdf/my_robot.xacro (robot description, xacro)
@@ -1,4 +1,5 @@
 <?xml version='1.0'?>
 <robot name="my_robot" xmlns:xacro="http://www.ros.org/wiki/xacro">
+<xacro:include filename="$(find my_robot)/urdf/my_robot.gazebo"/>
   <link name="robot_footprint"></link>
   <!-- Joint FootPrint-Chassis -->
@@ -201,8 +202,8 @@
   </gazebo>
   <gazebo reference="chassis">
-    <material>Gazebo/Indigo</material>
+    <material>Gazebo/SkyBlue</material>
   </gazebo>
   <gazebo reference="camera">
-    <material>Gazebo/FlatBlack</material>
+    <material>Gazebo/DarkGrey</material>
   </gazebo>
   <!-- End of the color configuration -->

Commit message: Add rviz configuration and joint_state_publisher

File: my_robot/urdf/my_robot.xacro (robot description, xacro)
@@ -24,5 +24,5 @@
   </joint>
   <!-- Joint Chassis-LeftWheel -->
-  <joint type="continuous" name="left_wheel_hinge">
+  <joint name="left_wheel_hinge" type="continuous">
     <origin xyz="0 0.15 0" rpy="0 0 0"/>
     <parent link="chassis"/>
@@ -33,5 +33,5 @@
   </joint>
   <!-- Joint Chassis-RightWheel -->
-  <joint type="continuous" name="right_wheel_hinge">
+  <joint name="right_wheel_hinge" type="continuous">
     <origin xyz="0 -0.15 0" rpy="0 0 0"/>
     <parent link="chassis"/>

Commit message: mapping node and RGBD camera

File: my_robot/urdf/my_robot.xacro (robot description, xacro)
@@ -41,4 +41,10 @@
     <dynamics damping="1.0" friction="1.0"/>
   </joint>
+  <!-- Joint RGBD camera -->
+  <joint name="camera_optical_joint" type="fixed">
+    <origin xyz="0 0 0" rpy="-1.5707 0 -1.5707"/>
+    <parent link="camera"/>
+    <child link="camera_link_optical"/>
+  </joint>
   <!-- Chassis -->
   <link name='chassis'>
@@ -194,4 +200,7 @@
   </link>
   <!-- End of the Hokuyo -->
+  <!-- RGBD camera -->
+  <link name="camera_link_optical">
+  </link>
   <!-- Color configuration -->
   <gazebo reference="left_wheel">

Commit message: Map my world to create my MAP

File: my_robot/urdf/my_robot.xacro (robot description, xacro)
@@ -19,4 +19,5 @@
   <joint name="camera_optical_joint" type="fixed">
     <origin xyz="0 0 0" rpy="-1.5707 0 -1.5707"/>
+<!--    <origin xyz="0 0 0" rpy="0 0 0"/> -->
     <parent link="camera"/>
     <child link="camera_link_optical"/>
